Commit message: added launchable box with camera

File: urdf/biosentry/box.urdf.xacro (robot description, xacro)
@@ -17,5 +17,5 @@
     </collision>
   </link>
-  <link name="base_motor">
+  <link name="inertia">
       <visual>
       <geometry>
@@ -29,9 +29,9 @@
     </inertial>
   </link>
-  <joint name="base_to_motor" type="fixed">
+  <joint name="base_to_inertia" type="fixed">
     <parent link="base_link"/>
-    <child link="base_motor"/>
+    <child link="inertia"/>
   </joint>
-    <!-- Gazebo plugin for ROS Control -->
+  <!-- Gazebo plugin for ROS Control -->
   <gazebo>
     <plugin name="gazebo_ros_control" filename="libgazebo_ros_control.so">
@@ -39,12 +39,3 @@
     </plugin>
   </gazebo>
-  <transmission name="sim_motor_trans">
-    <type>transmission_interface/SimpleTransmission</type>
-    <actuator name="sim_motor">
-      <mechanicalReduction>1</mechanicalReduction>
-    </actuator>
-    <joint name="base_to_motor">
-      <hardwareInterface>hardware_interface/VelocityJointInterface</hardwareInterface>
-    </joint>
-  </transmission>
 </robot>

Commit message: fixed dimensions and on box and added camera

File: urdf/biosentry/box.urdf.xacro (robot description, xacro)
@@ -1,6 +1,6 @@
 <?xml version="1.0"?>
 <robot name="box">
-  <material name="gray">
-    <color rgba="0.5 0.5 0.5 1"/>
+  <material name="red">
+    <color rgba="1 0 0 1"/>
   </material>
   <link name="base_link">
@@ -9,5 +9,5 @@
         <box size="0.136 0.065 0.044"/>
       </geometry>
-      <material name="gray"/>
+      <material name="red"/>
     </visual>
      <collision>
@@ -22,4 +22,5 @@
         <box size="0.01 0.01 0.01"/>
       </geometry>
+      <material name="red"/>
     </visual>
     <inertial>

File: urdf/biosentry/box_with_camera.urdf.xacro (robot description, xacro)
@@ -1,15 +1,15 @@
 <?xml version="1.0"?>
-<robot name="box_with_camera" xmlns:xacro="http://ros.org/wiki/xacro">
-  <material name="gray">
-    <color rgba="0.5 0.5 0.5 1"/>
+<robot name="box" xmlns:xacro="http://ros.org/wiki/xacro">>
+  <!-- material definitions. -->
+  <material name="red">
+    <color rgba="1.0 0.0 0.0 1.0"/>
   </material>
-  <material name="red">
-    <color rgba="0.9 0 0 1"/>
-  </material>
-  <!-- sizes in m. -->
+  <xacro:property name="pi" value="3.1415" />
   <xacro:property name="body_length" value="0.136" />
-  <xacro:property name="body_width" value="0.65" />
-  <xacro:property name="body_height" value="0.44" />
-  <xacro:property name="camera_size" value="0.1" />
+  <xacro:property name="body_width" value="0.065" />
+  <xacro:property name="body_height" value="0.044" />
+  <xacro:property name="body" value="${body_length} ${body_width} ${body_height}"/>
+  <xacro:property name="off_ground" value="0, ${body_height/2} 0"/>
+  <xacro:property name="camera_size" value="0.035" />
   <xacro:property name="camera_offset_x" value="${body_length/2}"/>
   <xacro:property name="camera_offset_z" value="${body_height/2}"/>
@@ -18,7 +18,8 @@
 <!-- =========================== Base link and inertia link =========================== -->
   <link name="base_link">
+    <origin xyz="0.0 0.0 ${body_height/2}"/> <!-- should mean center of geometry? -->
     <visual>
       <geometry>
-        <box size="${body_length} ${body_width} ${body_height}"/>
+        <box size="${body}"/>
       </geometry>
       <material name="gray"/>
@@ -26,5 +27,5 @@
      <collision>
       <geometry>
-        <box size="${body_length} ${body_width} ${body_height}"/>
+        <box size="${body}"/>
       </geometry>
     </collision>
@@ -37,5 +38,5 @@
       <visual>
       <geometry>
-        <box size="${body_length} ${body_width} ${body_height}"/>
+        <box size="${body}"/>
       </geometry>
     </visual>
@@ -47,11 +48,12 @@
   </link>
   <!--  =========================== camera joint, link and gazebo-cam-sensor =========================== -->
-  <joint name="base_to_camera" type="fixed">
+  <joint name="gimbal_pitch" type="revolute">
+    <axis xyz="0 1 0"/>
     <parent link="base_link"/>
-    <child link="camera_link"/>
-    <axis xyz="0 0 0" rpy="0 0 0" />
-    <origin xyz="${camera_offset_x} 0 ${camera_offset_z}" rpy="0 0 0"/>
+    <child link="gimbal_link"/>
+    <origin xyz="${camera_offset_x} 0 ${camera_offset_z}" rpy="0 ${pi/4} 0"/>
+    <limit lower="${-(pi/2)}" upper="${pi/2}" effort="30" velocity="1.0"/>
   </joint>
-   <link name="camera_link">
+   <link name="gimbal_link">
       <collision>
         <origin xyz="0 0 0" rpy="0 0 0"/>
@@ -73,6 +75,6 @@
       </inertial>
     </link>
-  <gazebo reference="camera_link">
-    <sensor type="camera" name="camera1">
+  <gazebo reference="gimbal_link">
+    <sensor type="camera" name="camera_front">
       <update_rate>30.0</update_rate>
       <camera name="head">
