Commit message: changed naming

File: urdf/biosentry/camera_box.urdf.xacro (robot description, xacro)
@@ -4,4 +4,8 @@
   <material name="red">
     <color rgba="1.0 0.0 0.0 1.0"/>
+  </material>
+    <!-- material definitions. -->
+  <material name="gray">
+    <color rgba="0.5 0.5 0.5 1.0"/>
   </material>
   <xacro:property name="pi" value="3.1415" />
